File: custom-flicker-LED.kicad_sch (KiCad schematic)
At the start: 8 parts, among them J1 TPI Interface, U1 ATtiny20-UU, U2 TL431DCK

Commit message: Update to show it working IRL, wooooo
Parts:
- R2: value 4.5kΩ -> 4.7kΩ
Changed lines of the file:
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@@
     (in_bom yes) (on_board yes)
     (property "Reference" "R2" (id 0) (at 161.925 86.1822 90))
-    (property "Value" "4.5kΩ" (id 1) (at 161.925 88.4936 90))
+    (property "Value" "4.7kΩ" (id 1) (at 161.925 88.4936 90))
     (property "Footprint" "Resistor_SMD:R_0402_1005Metric" (id 2) (at 161.925 89.662 90)
       (effects (font (size 1.27 1.27)) hide)
@@
     )
     (path "/8a0125f6-f8f3-4dd5-b01f-4d1c5ffe7675"
-      (reference "R2") (unit 1) (value "4.5kΩ") (footprint "Resistor_SMD:R_0402_1005Metric")
+      (reference "R2") (unit 1) (value "4.7kΩ") (footprint "Resistor_SMD:R_0402_1005Metric")
     )
     (path "/00000000-0000-0000-0000-00006230567c"
